Commit message: feat: upgrade Mengu to 6DoF, update ros2_control, add MoveIt config and Euler-Quaternion conversion service

File: src/mengu_description/urdf/mengu.urdf.xacro (robot description, xacro)
@@ -1,4 +1,4 @@
-<?xml version="1.0"?>
-<robot xmlns:xacro="http://www.ros.org/wiki/xacro" name="mengu">
+<?xml version="1.0" encoding="utf-8"?>
+<robot xmlns:xacro="http://wiki.ros.org/xacro" name="mengu">
     <xacro:arg name="is_ignition" default="true"/>
     <xacro:include filename="$(find mengu_description)/urdf/mengu_gazebo.xacro" />
@@ -7,197 +7,230 @@
     <xacro:property name="effort" value="30.0" />
     <xacro:property name="velocity" value="10.0" />
-    <xacro:macro name="default_inertial" params="mass">
-        <inertial>
-            <mass value="${mass}"/>
-            <inertia ixx="1.0" ixy="0.0" ixz="0.0" iyy="1.0" iyz="0.0" izz="1.0"/>
-        </inertial>
-    </xacro:macro>
+    <xacro:arg name="limit_angles" default="$(find mengu_controller)/config/mengu_parameters.yaml" />
+    <xacro:property name="limits" value="${xacro.load_yaml('$(arg limit_angles)')}" />
     <material name="blue">
-        <color rgba="0 0 1 1" />
+        <color rgba="0 0 1 1"/>
     </material>
-    <link name="world" />
+    <!-- WORLD -->
+     <link name="world"/>
+    <!--VIRTUAL JOINT-->
+    <joint name="virtual_joint" type="fixed">
+        <parent link="world"/>
+        <child link="base_link"/>
+    </joint>
     <link name="base_link">
-        <xacro:default_inertial mass="1.0" />
-        <visual>
-            <material name="blue" />
-            <origin rpy="0 0 0" xyz="-0.5 -0.5 0" />
-            <geometry>
-                <mesh filename="package://mengu_description/meshes/basement.STL" scale="0.01 0.01 0.01" />
-            </geometry>
-        </visual>
-        <collision>
-            <origin rpy="0 0 0" xyz="-0.5 -0.5 0" />
-            <geometry>
-                <mesh filename="package://mengu_description/meshes/basement.STL" scale="0.01 0.01 0.01" />
-            </geometry>
-        </collision>
-    </link>
-    <joint name="virtual_joint" type="fixed">
-        <parent link="world" />
-        <child link="base_link" />
-        <origin rpy="0 0 0" xyz="0 0 0" />
-    </joint>
-    <link name="base_plate">
-        <xacro:default_inertial mass="0.1" />
-        <visual>
-            <origin rpy="0 0 0" xyz="-0.39 -0.39 -0.56" />
-            <geometry>
-                <mesh filename="package://mengu_description/meshes/base_plate.STL" scale="0.01 0.01 0.01" />
-            </geometry>
-        </visual>
-        <collision>
-            <origin rpy="0 0 0" xyz="-0.39 -0.39 -0.56" />
-            <geometry>
-                <mesh filename="package://mengu_description/meshes/base_plate.STL" scale="0.01 0.01 0.01" />
-            </geometry>
-        </collision>
+      <inertial>
+        <origin rpy="0 0 0" xyz="0 0 0"/>
+        <mass value="0.7102"/>
+        <inertia ixx="0.0039943" ixy="3.697E-07" ixz="-5.7364E-08"
+                 iyy="0.0014946" iyz="-0.00036051" izz="0.0042554"/>
+      </inertial>
+      <visual>
+        <origin rpy="0 0 0" xyz="0 0 0"/>
+        <geometry>
+            <mesh filename="package://mengu_description/meshes/base_link.STL"/>
+        </geometry>
+      </visual>
+      <collision>
+        <origin rpy="0 0 0" xyz="0 0 0"/>
+        <geometry>
+            <mesh filename="package://mengu_description/meshes/base_link.STL"/>
+        </geometry>
+      </collision>
+    </link>
+    <link name="link_1">
+      <inertial>
+        <origin rpy="0 0 0" xyz="0 0 0"/>
+        <mass value="0.88065"/>
+        <inertia ixx="0.0034" ixy="0.00042296" ixz="-0.00089231"
+                 iyy="0.0041778" iyz="0.0010848" izz="0.0027077"/>
+      </inertial>
+      <visual>
+        <material name="blue"/>
+        <origin xyz="0 0 -0.092" rpy="${-PI} 0 0"/>
+        <geometry>
+            <mesh filename="package://mengu_description/meshes/link_1.STL"/>
+        </geometry>
+      </visual>
+      <collision>
+        <origin xyz="0 0 0" rpy="0 0 0"/>
+        <geometry>
+            <mesh filename="package://mengu_description/meshes/link_1.STL"/>
+        </geometry>
+      </collision>
     </link>
     <joint name="joint_1" type="revolute">
-        <parent link="base_link"/>
-        <child link="base_plate"/>
-        <origin rpy="0 0 0" xyz="0 0 0.307" />
-        <axis xyz="0 0 1" />
-        <limit lower="-${PI/2}" upper="${PI/2}" effort="${effort}" velocity="${velocity}" />
-    </joint>
-    <link name="forward_drive_arm">
-        <xacro:default_inertial mass="0.1" />
-        <visual>
-            <material name="blue" />
-            <origin rpy="0 -${PI/2} ${PI/2}" xyz="0.19 0.06 -0.08" />
-            <geometry>
-                <mesh filename="package://mengu_description/meshes/forward_drive_arm.STL" scale="0.01 0.01 0.01"/>
-            </geometry>
-        </visual>
-        <collision>
-            <origin rpy="0 -${PI/2} ${PI/2}" xyz="0.19 0.06 -0.08" />
-            <geometry>
-                <mesh filename="package://mengu_description/meshes/forward_drive_arm.STL" scale="0.01 0.01 0.01"/>
-            </geometry>
-        </collision>
+      <origin rpy="0 0 0" xyz="0 0 0.092"/>
+      <parent link="base_link"/>
+      <child link="link_1"/>
+      <axis xyz="0 0 1"/>
+      <limit
+        lower="${limits['j1_min']}"
+        upper="${limits['j1_max']}"
+        effort="100"
+        velocity="1.0472"
+      />
+    </joint>
+    <link name="link_2">
+      <inertial>
+        <origin rpy="0 0 0" xyz="0 0 0"/>
+        <mass value="0.57738"/>
+        <inertia ixx="0.0047312" ixy="0.0022624" ixz="0.00032144"
+                 iyy="0.0020836" iyz="-0.00056569" izz="0.0056129"/>
+      </inertial>
+      <visual>
+        <origin xyz="0 0 0" rpy="0 0 ${-PI}"/>
+        <geometry>
+            <mesh filename="package://mengu_description/meshes/link_2.STL"/>
+        </geometry>
+      </visual>
+      <collision>
+        <origin xyz="0 0 0" rpy="0 0 0"/>
+        <geometry>
+            <mesh filename="package://mengu_description/meshes/link_2.STL"/>
+        </geometry>
+      </collision>
     </link>
     <joint name="joint_2" type="revolute">
-        <parent link="base_plate"/>
-        <child link="forward_drive_arm"/>
-        <origin rpy="0 0 0" xyz="-0.02 0 0.35" />
-        <axis xyz="1 0 0"/>
-        <limit lower="-${PI/2}" upper="${PI/2}" effort="${effort}" velocity="${velocity}"/>
-    </joint>
-    <link name="horizontal_arm">
-        <xacro:default_inertial mass="0.1" />
-        <visual>
-            <origin rpy="${PI/2} 0 ${PI/2}" xyz="-0.03 -0.4 -0.06" />
-            <geometry>
-                <mesh filename="package://mengu_description/meshes/horizontal_arm.STL" scale="0.01 0.01 0.01"/>
-            </geometry>
-        </visual>
-        <collision>
-            <origin rpy="${PI/2} 0 ${PI/2}" xyz="-0.03 -0.4 -0.06" />
-            <geometry>
-                <mesh filename="package://mengu_description/meshes/horizontal_arm.STL" scale="0.01 0.01 0.01"/>
-            </geometry>
-        </collision>
+      <origin rpy="1.5708 0 -1.5708" xyz="0 -0.06415 0.07778"/>
+      <parent link="link_1"/>
+      <child link="link_2"/>
+      <axis xyz="0 0 -1"/>
+      <limit
+        lower="${limits['j2_min']}"
+        upper="${limits['j2_max']}"
+        effort="100"
+        velocity="1.0472"
+      />
+    </joint>
+    <link name="link_3">
+      <inertial>
+        <origin rpy="0 0 0" xyz="-0.00029765 -0.023661 -0.0019125"/>
+        <mass value="0.1787"/>
+        <inertia ixx="0.0001685" ixy="-2.7713E-05" ixz="5.6885E-06"
+                 iyy="0.00012865" iyz="2.9256E-05" izz="0.00020744"/>
+      </inertial>
+      <visual>
+        <material name="blue"/>
+        <origin xyz="0 0 0" rpy="0 0 0 "/>
+        <geometry>
+            <mesh filename="package://mengu_description/meshes/link_3.STL"/>
+        </geometry>
+      </visual>
+      <collision>
+        <origin xyz="0 0 0" rpy="0 0 0"/>
+        <geometry>
+            <mesh filename="package://mengu_description/meshes/link_3.STL"/>
+        </geometry>
+      </collision>
     </link>
     <joint name="joint_3" type="revolute">
-        <parent link="forward_drive_arm" />
-        <child link="horizontal_arm" />
-        <axis xyz="1 0 0"/>
-        <origin rpy="0 0 0" xyz="0 0 0.8"/>
-        <limit lower="-${PI/2}" upper="${PI/2}" effort="${effort}" velocity="${velocity}"/>
-    </joint>
-    <link name="claw_support">
-        <xacro:default_inertial mass="0.05" />
-        <visual>
-            <origin rpy="0 0 ${PI / 2}" xyz="0 -0.05 -0.15"/>
-            <geometry>
-                <mesh filename="package://mengu_description/meshes/claw_support.STL" scale="0.01 0.01 0.01"/>
-            </geometry>
-        </visual>
-        <collision>
-            <origin rpy="0 0 ${PI / 2}" xyz="0 -0.05 -0.15"/>
-            <geometry>
-                <mesh filename="package://mengu_description/meshes/claw_support.STL" scale="0.01 0.01 0.01"/>
-            </geometry>
-        </collision>
-    </link>
-    <joint name="horizontal_arm_to_claw_support" type="fixed">
-        <parent link="horizontal_arm"/>
-        <child link="claw_support"/>
-        <origin rpy="0 0 0" xyz="0 0.82 0"/>
-    </joint>
-    <link name="gripper_right">
-        <xacro:default_inertial mass="0.01" />
-        <visual>
-            <material name="blue"/>
-            <origin rpy="0 0 -${PI / 2}" xyz="-0.1 0.50 -0.1"/>
-            <geometry>
-                <mesh filename="package://mengu_description/meshes/right_finger.STL" scale="0.01 0.01 0.01"/>
-            </geometry>
-        </visual>
-        <collision>
-            <origin rpy="0 0 -${PI / 2}" xyz="-0.1 0.50 -0.1"/>
-            <geometry>
-                <mesh filename="package://mengu_description/meshes/right_finger.STL" scale="0.01 0.01 0.01"/>
-            </geometry>
-        </collision>
-    </link>
-    <link name="gripper_left">
-        <xacro:default_inertial mass="0.01" />
-        <visual>
-            <material name="blue"/>
-            <origin rpy="0 0 -${PI / 2}" xyz="-0.04 0.50 -0.1"/>
-            <geometry>
-                <mesh filename="package://mengu_description/meshes/left_finger.STL" scale="0.01 0.01 0.01"/>
-            </geometry>
-        </visual>
-        <collision>
-            <origin rpy="0 0 -${PI / 2}" xyz="-0.04 0.50 -0.1"/>
-            <geometry>
-                <mesh filename="package://mengu_description/meshes/left_finger.STL" scale="0.01 0.01 0.01"/>
-            </geometry>
-        </collision>
-    </link>
-    <joint name ="joint_4" type="revolute">
-        <parent link="claw_support"/>
-        <child link = "gripper_right"/>
-        <origin xyz="-0.04 0.13 -0.1"/>
-        <axis xyz="0 0 1"/>
-        <limit lower="-${PI / 2}" upper="0.0"
-               effort="${effort}" velocity="${velocity}"/>
-    </joint>
-    <joint name ="joint_5" type="revolute">
-        <parent link="claw_support"/>
-        <child link = "gripper_left"/>
-        <origin xyz="-0.22 0.13 -0.1"/>
-        <axis xyz="0 0 1"/>
-        <limit lower="0.0" upper="${PI / 2}"
-               effort="${effort}" velocity="${velocity}"/>
-        <mimic joint="joint_4" multiplier="-1"/>
-    </joint>
-    <link name="rgb_camera">
-        <visual>
-            <xacro:default_inertial mass="0.001" />
-            <origin rpy="-1.57 0 -1.57" xyz="-0.1 0.125 0.15"/>
-            <geometry>
-                <mesh filename="package://mengu_description/meshes/pi_camera.STL" scale="0.01 0.01 0.01"/>
-            </geometry>
-        </visual>
-        <collision>
-            <origin rpy="-1.57 0 -1.57" xyz="-0.1 0.125 0.15"/>
-            <geometry>
-                <mesh filename="package://mengu_description/meshes/pi_camera.STL" scale="0.01 0.01 0.01"/>
-            </geometry>
-        </collision>
-    </link>
-    <joint name ="rgb_camera_joint" type="fixed">
-        <parent link="base_link"/>
-        <child link = "rgb_camera"/>
-        <origin xyz="0 0.45 0.2" rpy="0 -0.5 1.57"/>
-    </joint>
-    <gazebo>
-        <plugin name="mimic_plugin" filename="libgazebo_ros_joint_pose_plugin.so">
-            <joint_name>joint_5</joint_name>
-            <parent_joint_name>joint_4</parent_joint_name>
-            <multiplier>-1</multiplier>
-        </plugin>
-    </gazebo>
+      <origin rpy="0 0 3.1416" xyz="0 0.305 0.007"/>
+      <parent link="link_2"/>
+      <child link="link_3"/>
+      <axis xyz="0 0 -1"/>
+      <limit
+        lower="${limits['j3_min']}"
+        upper="${limits['j3_max']}"
+        effort="100"
+        velocity="1.0472"
+      />
+    </joint>
+    <link name="link_4">
+      <inertial>
+        <origin rpy="0 0 0" xyz="-0.0016798 -0.00057319 -0.074404"/>
+        <mass value="0.34936"/>
+        <inertia ixx="0.0030532" ixy="-1.8615E-05" ixz="-7.0047E-05"
+                 iyy="0.0031033" iyz="-2.3301E-05" izz="0.00022264"/>
+      </inertial>
+      <visual>
+        <origin xyz="0 0 0" rpy="0 0 0 "/>
+        <geometry>
+            <mesh filename="package://mengu_description/meshes/link_4.STL"/>
+        </geometry>
+      </visual>
+      <collision>
+        <origin xyz="0 0 0" rpy="0 0 0"/>
+        <geometry>
+            <mesh filename="package://mengu_description/meshes/link_4.STL"/>
+        </geometry>
+      </collision>
+    </link>
+    <joint name="joint_4" type="revolute">
+      <origin rpy="1.5708 0 -1.5708" xyz="0 0 0"/>
+      <parent link="link_3"/>
+      <child link="link_4"/>
+      <axis xyz="0 0 -1"/>
+      <limit
+        lower="${limits['j4_min']}"
+        upper="${limits['j4_max']}"
+        effort="100"
+        velocity="1.0472"
+      />
+    </joint>
+    <link name="link_5">
+      <inertial>
+        <origin rpy="0 0 0" xyz="0.0015066 -1.3102E-05 -0.012585"/>
+        <mass value="0.11562"/>
+        <inertia ixx="5.5035E-05" ixy="-1.019E-08" ixz="-2.6243E-06"
+                 iyy="8.2921E-05" iyz="1.4437E-08" izz="5.2518E-05"/>
+      </inertial>
+      <visual>
+        <material name="blue"/>
+        <origin xyz="0 0 0" rpy="0 0 0"/>
+        <geometry>
+            <mesh filename="package://mengu_description/meshes/link_5.STL"/>
+        </geometry>
+      </visual>
+      <collision>
+        <origin xyz="0 0 0" rpy="0 0 0"/>
+        <geometry>
+            <mesh filename="package://mengu_description/meshes/link_5.STL"/>
+        </geometry>
+      </collision>
+    </link>
+    <joint name="joint_5" type="revolute">
+      <origin rpy="${PI} 0 -1.5708" xyz="0 0 -0.22294"/>
+      <parent link="link_4"/>
+      <child link="link_5"/>
+      <axis xyz="1 0 0"/>
+      <limit
+        lower="${limits['j5_min']}"
+        upper="${limits['j5_max']}"
+        effort="100"
+        velocity="1.0472"
+      />
+    </joint>
+    <link name="link_6">
+      <inertial>
+        <origin rpy="0 0 0" xyz="2.9287E-10 -1.6472E-09 0.0091432"/>
+        <mass value="0.013863"/>
+        <inertia ixx="1.3596E-06" ixy="3.0585E-13" ixz="5.7102E-14"
+                 iyy="1.7157E-06" iyz="6.3369E-09" izz="2.4332E-06"/>
+      </inertial>
+      <visual>
+        <origin xyz="0 0 0" rpy="0 0 0"/>
+        <geometry>
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
File: src/mengu_description/urdf/mengu_gazebo.xacro (robot description, xacro)
@@ -3,8 +3,7 @@
   <!-- ROS 2 Control -->
   <gazebo>
-    <!-- ROS 2 Iron or above -->
     <xacro:unless value="$(arg is_ignition)">
       <plugin filename="gz_ros2_control-system" name="gz_ros2_control::GazeboSimROS2ControlPlugin">
-	<parameters>$(find mengu_controller)/config/mengu_controllers.yaml</parameters>
+        <parameters>$(find mengu_controller)/config/mengu_controllers.yaml</parameters>
       </plugin>
     </xacro:unless>

File: src/mengu_description/urdf/mengu_ros2_control.xacro (robot description, xacro)
@@ -2,7 +2,6 @@
 <robot xmlns:xacro="http://www.ros.org/wiki/xacro" name="mengu">
     <ros2_control name="RobotSystem" type="system">
-        <xacro:property name="PI" value="3.14159265359" />
-        <!-- ros2_control Gazebo -->
-        <!-- ROS 2 Iron or above -->
+        <xacro:arg name="limit_angles" default="$(find mengu_controller)/config/mengu_parameters.yaml" />
+        <xacro:property name="limits" value="${xacro.load_yaml('$(arg limit_angles)')}" />
         <xacro:unless value="$(arg is_ignition)">
             <hardware>
@@ -12,6 +11,6 @@
         <joint name="joint_1">
             <command_interface name="position">
-            <param name="min">-${PI / 2}</param>
-            <param name="max">${PI / 2}</param>
+                <param name="min">${limits['j1_min']}</param>
+                <param name="max">${limits['j1_max']}</param>
             </command_interface>
             <state_interface name="position"/>
@@ -19,6 +18,6 @@
         <joint name="joint_2">
             <command_interface name="position">
-            <param name="min">-${PI / 2}</param>
-            <param name="max">${PI / 2}</param>
+                <param name="min">${limits['j2_min']}</param>
+                <param name="max">${limits['j2_max']}</param>
             </command_interface>
             <state_interface name="position"/>
@@ -26,6 +25,6 @@
         <joint name="joint_3">
             <command_interface name="position">
-            <param name="min">-${PI / 2}</param>
-            <param name="max">${PI / 2}</param>
+                <param name="min">${limits['j3_min']}</param>
+                <param name="max">${limits['j3_max']}</param>
             </command_interface>
             <state_interface name="position"/>
@@ -33,12 +32,22 @@
         <joint name="joint_4">
             <command_interface name="position">
-            <param name="min">-${PI / 2}</param>
-            <param name="max">0.0</param>
+                <param name="min">${limits['j4_min']}</param>
+                <param name="max">${limits['j4_max']}</param>
             </command_interface>
             <state_interface name="position"/>
         </joint>
         <joint name="joint_5">
-            <param name="mimic">joint_4</param>
-            <param name="multiplier">-1</param>
+            <command_interface name="position">
+                <param name="min">${limits['j5_min']}</param>
+                <param name="max">${limits['j5_max']}</param>
+            </command_interface>
+            <state_interface name="position"/>
+        </joint>
+        <joint name="joint_6">
+            <command_interface name="position">
+                <param name="min">${limits['j6_min']}</param>
+                <param name="max">${limits['j6_max']}</param>
+            </command_interface>
+            <state_interface name="position"/>
         </joint>
     </ros2_control>
