Commit message: Complete MoveIt configuration and performance fixes

File: src/mengu_description/urdf/mengu.urdf.xacro (robot description, xacro)
@@ -10,5 +10,8 @@
     <xacro:property name="limits" value="${xacro.load_yaml('$(arg limit_angles)')}" />
     <material name="blue">
-        <color rgba="0 0 1 1"/>
+        <color rgba="0 0 0.65 1"/>
+    </material>
+    <material name="gray">
+      <color rgba="0.5 0.5 0.5 1"/>
     </material>
     <!-- WORLD -->
@@ -27,4 +30,6 @@
       </inertial>
       <visual>
+        <material name="gray"/>
+        <material>Gazebo/BrushedMetal</material>
         <origin rpy="0 0 0" xyz="0 0 0"/>
         <geometry>
@@ -48,4 +53,13 @@
       <visual>
         <material name="blue"/>
+        <material>
+          <pbr>
+            <metal>
+              <albedo>0.3 0.3 0.3 1</albedo>
+              <metalness>0.9</metalness>
+              <roughness>0.4</roughness>
+            </metal>
+          </pbr>
+        </material>
         <origin xyz="0 0 -0.092" rpy="${-PI} 0 0"/>
         <geometry>
@@ -56,5 +70,5 @@
         <origin xyz="0 0 0" rpy="0 0 0"/>
         <geometry>
-            <mesh filename="package://mengu_description/meshes/link_1.STL"/>
+            <cylinder radius="0.02" length="0.05"/>
         </geometry>
       </collision>
@@ -68,5 +82,5 @@
         lower="${limits['j1_min']}"
         upper="${limits['j1_max']}"
-        effort="100"
+        effort="1000"
         velocity="1.0472"
       />
@@ -80,4 +94,6 @@
       </inertial>
       <visual>
+        <material name="gray"/>
+        <material>Gazebo/BrushedMetal</material>
         <origin xyz="0 0 0" rpy="0 0 ${-PI}"/>
         <geometry>
@@ -88,5 +104,5 @@
         <origin xyz="0 0 0" rpy="0 0 0"/>
         <geometry>
-            <mesh filename="package://mengu_description/meshes/link_2.STL"/>
+            <cylinder radius="0.02" length="0.05"/>
         </geometry>
       </collision>
@@ -100,5 +116,5 @@
         lower="${limits['j2_min']}"
         upper="${limits['j2_max']}"
-        effort="100"
+        effort="1000"
         velocity="1.0472"
       />
@@ -113,4 +129,5 @@
       <visual>
         <material name="blue"/>
+        <material>Gazebo/BrushedMetal</material>
         <origin xyz="0 0 0" rpy="0 0 0 "/>
         <geometry>
@@ -121,5 +138,5 @@
         <origin xyz="0 0 0" rpy="0 0 0"/>
         <geometry>
-            <mesh filename="package://mengu_description/meshes/link_3.STL"/>
+            <cylinder radius="0.02" length="0.05"/>
         </geometry>
       </collision>
@@ -133,5 +150,5 @@
         lower="${limits['j3_min']}"
         upper="${limits['j3_max']}"
-        effort="100"
+        effort="1000"
         velocity="1.0472"
       />
@@ -145,4 +162,6 @@
       </inertial>
       <visual>
+        <material name="gray"/>
+        <material>Gazebo/BrushedMetal</material>
         <origin xyz="0 0 0" rpy="0 0 0 "/>
         <geometry>
@@ -153,5 +172,5 @@
         <origin xyz="0 0 0" rpy="0 0 0"/>
         <geometry>
-            <mesh filename="package://mengu_description/meshes/link_4.STL"/>
+            <cylinder radius="0.02" length="0.05"/>
         </geometry>
       </collision>
@@ -165,5 +184,5 @@
         lower="${limits['j4_min']}"
         upper="${limits['j4_max']}"
-        effort="100"
+        effort="1000"
         velocity="1.0472"
       />
@@ -178,4 +197,5 @@
       <visual>
         <material name="blue"/>
+        <material>Gazebo/BrushedMetal</material>
         <origin xyz="0 0 0" rpy="0 0 0"/>
         <geometry>
@@ -186,5 +206,5 @@
         <origin xyz="0 0 0" rpy="0 0 0"/>
         <geometry>
-            <mesh filename="package://mengu_description/meshes/link_5.STL"/>
+            <cylinder radius="0.02" length="0.05"/>
         </geometry>
       </collision>
@@ -198,5 +218,5 @@
         lower="${limits['j5_min']}"
         upper="${limits['j5_max']}"
-        effort="100"
+        effort="1000"
         velocity="1.0472"
       />
@@ -210,4 +230,6 @@
       </inertial>
       <visual>
+        <material name="gray"/>
+        <material>Gazebo/BrushedMetal</material>
         <origin xyz="0 0 0" rpy="0 0 0"/>
         <geometry>
@@ -218,5 +240,5 @@
         <origin xyz="0 0 0" rpy="0 0 0"/>
         <geometry>
-            <mesh filename="package://mengu_description/meshes/link_6.STL"/>
+            <cylinder radius="0.02" length="0.05"/>
         </geometry>
       </collision>
@@ -230,5 +252,5 @@
         lower="${limits['j6_min']}"
         upper="${limits['j6_max']}"
-        effort="100"
+        effort="1000"
         velocity="1.5708"
       />
